File: Hardware/demonBoard/demonBoard.kicad_sch (KiCad schematic)
At the start: 0 parts

Commit message: doc: Add schematic pdf
Other:
- company: mangoByte -> Vagarth Gaurav
Changed lines of the file:
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@@
 	(title_block
 		(title "Demon board")
-		(rev "0.1")
-		(company "mangoByte")
+		(date "2026-01-05")
+		(company "Vagarth Gaurav")
 	)
 	(text "DEMON BOARD"
