File: Hardware/demonBoard/voltage_regulators_and_voltage_sense.kicad_sch (KiCad schematic)
At the start: 35 parts, among them U6 TPS61288, U7 TPS563201

Commit message: doc: Add schematic pdf
Other:
- company: (none) -> Vagarth Gaurav
- title: (none) -> Demon board
- moved on the sheet: C14, C15, C16, C17, C18, C19, C20, C21, C22, C23, C24, C25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

Commit message: feat: Add ibom.html
Parts:
- C16, C17: value 22u -> 22u/25V
Changed lines of the file:
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@@
 			)
 		)
-		(property "Value" "22u"
+		(property "Value" "22u/25V"
 			(at 145.796 101.6 0)
 			(effects
@@
 			)
 		)
-		(property "Value" "22u"
+		(property "Value" "22u/25V"
 			(at 135.636 101.6 0)
 			(effects

Commit message: Change resistors for leds
Parts:
- C24: now fitted
- R15, R20: value 1k -> 10k
Changed lines of the file:
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@@
 			)
 		)
-		(property "Value" "1k"
+		(property "Value" "10k"
 			(at 303.784 221.234 0)
 			(effects
@@
 			)
 		)
-		(property "Value" "1k"
+		(property "Value" "10k"
 			(at 307.594 104.394 0)
 			(effects
@@
 		(in_bom yes)
 		(on_board yes)
-		(dnp yes)
+		(dnp no)
 		(property "Reference" "C24"
 			(at 297.942 98.044 0)
