File: Hardware/demonSpawn/demonSpawn.kicad_sch (KiCad schematic)
At the start: 0 parts

Commit message: doc: Add schematic pdf
Other:
- company: (none) -> Vagarth Gaurav
- title: (none) -> Demon Spawn Remote
Changed lines of the file:
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@@
 	(generator_version "9.0")
 	(paper "A4")
+	(title_block
+		(title "Demon Spawn Remote")
+		(date "2026-01-05")
+		(company "Vagarth Gaurav")
+	)
 	(text "Demon spawn remote"
 		(exclude_from_sim no)
