File: Hardware/demonSpawn/microcontroller.kicad_sch (KiCad schematic)
At the start: 25 parts, among them U2 ESP32-C3-WROOM-02, U3 SPX3819M5-L-3-3

Commit message: doc: Add schematic pdf
Changed lines of the file:
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@@
+		)
+	)
+	(polyline
+		(pts
+			(xy 128.27 21.59) (xy 186.69 21.59)
+		)
+		(stroke
+			(width 0.5)
+			(type solid)
 		)
 	)
